File: L1/L1.kicad_pcb (KiCad board)
At the start: 2 copper layers, 264 x 32 mm, 1 part

Commit message: Add kicad projects for PCB build
Parts:
- removed the REF** at (16.7, 60.8)
- added REF**: CIS_Edge_1, CIS:CIS_Edge_Holes, F.Cu at (16.6, 125.0)
- added REF**: CIS_Edge_1, CIS:CIS_Edge_L1, F.Cu at (16.6, 125.0)
Routing:
- removed copper zone on F.Cu, net (none)
Changed lines of the file:
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@@
     (39 "F.Mask" user)
     (40 "Dwgs.User" user "User.Drawings")
+    (41 "Cmts.User" user "User.Comments")
     (42 "Eco1.User" user "User.Eco1")
     (43 "Eco2.User" user "User.Eco2")
@@
     (48 "B.Fab" user)
     (49 "F.Fab" user)
+    (50 "User.1" user)
+    (51 "User.2" user)
+    (52 "User.3" user)
+    (53 "User.4" user)
+    (54 "User.5" user)
+    (55 "User.6" user)
+    (56 "User.7" user)
+    (57 "User.8" user)
+    (58 "User.9" user)
   )
   (setup
     (stackup
-      (layer "F.SilkS" (type "Top Silk Screen"))
+      (layer "F.SilkS" (type "Top Silk Screen") (color "White"))
       (layer "F.Paste" (type "Top Solder Paste"))
       (layer "F.Mask" (type "Top Solder Mask") (color "Black") (thickness 0.01))
@@
       (layer "B.Mask" (type "Bottom Solder Mask") (color "Black") (thickness 0.01))
       (layer "B.Paste" (type "Bottom Solder Paste"))
-      (layer "B.SilkS" (type "Bottom Silk Screen"))
-      (copper_finish "HAL lead-free")
+      (layer "B.SilkS" (type "Bottom Silk Screen") (color "White"))
+      (copper_finish "None")
       (dielectric_constraints no)
-      (castellated_pads yes)
-      (edge_plating yes)
     )
     (pad_to_mask_clearance 0)
-    (aux_axis_origin 17.3 112.8)
-    (grid_origin 17.3 112.8)
+    (aux_axis_origin 16.62132 125)
+    (grid_origin 16.62132 125)
     (pcbplotparams
-      (layerselection 0x00010cc_ffffffff)
+      (layerselection 0x00010fc_ffffffff)
       (disableapertmacros false)
       (usegerberextensions false)
@@
       (outputformat 1)
       (mirror false)
-      (drillshape 0)
+      (drillshape 1)
       (scaleselection 1)
-      (outputdirectory "Gerber/")
+      (outputdirectory "")
     )
   )
   (net 0 "")
-  (footprint "Library:CIS_Edge_1" (layer "F.Cu")
-    (at 16.700001 60.8)
-    (attr through_hole)
+  (footprint "CIS:CIS_Edge_Holes" (layer "F.Cu")
+    (at 16.62132 125)
+    (attr through_hole board_only exclude_from_pos_files exclude_from_bom)
     (fp_text reference "REF**" (at 0.05 7 unlocked) (layer "F.SilkS") hide
       (effects (font (size 1 1) (thickness 0.15)))
     )
-    (fp_text value "CIS_Edge_1" (at 0 6.9 unlocked) (layer "F.Fab")
+    (fp_text value "CIS_Edge_1" (at 0 6.9 unlocked) (layer "F.Fab") hide
       (effects (font (size 1 1) (thickness 0.15)))
     )
-    (fp_line (start 0 -3) (end 0 -29) (layer "B.Mask") (width 3))
-    (fp_line (start 3 -32) (end 261 -32) (layer "B.Mask") (width 3))
-    (fp_line (start 261 0) (end 3 0) (layer "B.Mask") (width 3))
-    (fp_line (start 264 -29) (end 264 -3) (layer "B.Mask") (width 3))
-    (fp_arc (start 0 -29) (mid 0.878686 -31.121314) (end 3 -32) (layer "B.Mask") (width 3))
-    (fp_arc (start 3 0) (mid 0.878694 -0.878694) (end 0 -3) (layer "B.Mask") (width 3))
-    (fp_arc (start 261 -32) (mid 263.12132 -31.12132) (end 264 -29) (layer "B.Mask") (width 3))
-    (fp_arc (start 264 -3) (mid 263.12132 -0.87868) (end 261 0) (layer "B.Mask") (width 3))
-    (fp_line (start -0.000001 -28.999999) (end -0.000001 -2.999999) (layer "F.Mask") (width 3))
-    (fp_line (start 260.999999 -31.999999) (end 2.999999 -31.999999) (layer "F.Mask") (width 3))
-    (fp_line (start 263.999999 -2.999999) (end 263.999999 -28.999999) (layer "F.Mask") (width 3))
-    (fp_line (start 2.999999 0.000001) (end 260.999999 0.000001) (layer "F.Mask") (width 3))
-    (fp_arc (start 2.999999 0.000001) (mid 0.878679 -0.878679) (end -0.000001 -2.999999) (layer "F.Mask") (width 3))
-    (fp_arc (start 263.999999 -2.999999) (mid 263.121319 -0.87868) (end 260.999999 0.000001) (layer "F.Mask") (width 3))
-    (fp_arc (start -0.000001 -28.999999) (mid 0.878679 -31.121319) (end 2.999999 -31.999999) (layer "F.Mask") (width 3))
-    (fp_arc (start 260.999999 -31.999999) (mid 263.12132 -31.12132) (end 263.999999 -28.999999) (layer "F.Mask") (width 3))
-    (fp_line (start 3 0) (end 261 0) (layer "Edge.Cuts") (width 1))
-    (fp_line (start 0 -29) (end 0 -3) (layer "Edge.Cuts") (width 1))
-    (fp_line (start 264 -3) (end 264 -29) (layer "Edge.Cuts") (width 1))
-    (fp_line (start 261 -32) (end 3 -32) (layer "Edge.Cuts") (width 1))
-    (fp_arc (start 0 -29) (mid 0.87868 -31.12132) (end 3 -32) (layer "Edge.Cuts") (width 1))
-    (fp_arc (start 264 -3) (mid 263.12132 -0.87868) (end 261 0) (layer "Edge.Cuts") (width 1))
-    (fp_arc (start 261 -32) (mid 263.12132 -31.12132) (end 264 -29) (layer "Edge.Cuts") (width 1))
-    (fp_arc (start 3 0) (mid 0.87868 -0.87868) (end 0 -3) (layer "Edge.Cuts") (width 1))
-    (pad "" thru_hole circle (at 88 -3.5) (size 3 3) (drill 2.2) (layers *.Cu *.Mask))
     (pad "" thru_hole circle (at 176 -3.5287) (size 3 3) (drill 2.2) (layers *.Cu *.Mask))
-    (pad "" thru_hole circle (at 176 -28.5) (size 3 3) (drill 2.2) (layers *.Cu *.Mask))
-    (pad "" thru_hole circle (at 260.5 -3.5) (size 3 3) (drill 2.2) (layers *.Cu *.Mask))
     (pad "" thru_hole circle (at 3.5 -3.5) (size 3 3) (drill 2.2) (layers *.Cu *.Mask))
+    (pad "" thru_hole circle (at 3.5 -28.5) (size 3 3) (drill 2.2) (layers *.Cu *.Mask))
     (pad "" thru_hole circle (at 260.5 -28.5) (size 3 3) (drill 2.2) (layers *.Cu *.Mask))
     (pad "" thru_hole circle (at 88 -28.5) (size 3 3) (drill 2.2) (layers *.Cu *.Mask))
-    (pad "" thru_hole circle (at 3.5 -28.5) (size 3 3) (drill 2.2) (layers *.Cu *.Mask))
-    (group "" (id 71bf3650-a719-42d3-adb1-1560e575cd5a)
+    (pad "" thru_hole circle (at 260.5 -3.5) (size 3 3) (drill 2.2) (layers *.Cu *.Mask))
+    (pad "" thru_hole circle (at 88 -3.5) (size 3 3) (drill 2.2) (layers *.Cu *.Mask))
+    (pad "" thru_hole circle (at 176 -28.5) (size 3 3) (drill 2.2) (layers *.Cu *.Mask))
+    (group "" (id f8577c47-52d4-4a5f-be8e-504480dca4de)
       (members
-        01bc44b6-94b0-4a26-ba01-24cbf4c91c2c
-        045825ae-fad3-492f-a879-f5de111e3e7a
-        0583167e-23bf-4146-854c-1ed6b4396f85
-        058bd0c5-8a31-4b7a-8b22-aae8da297c3f
-        1030d820-21bf-4dd8-9a24-13bfd1154c95
-        31d888b9-cf74-467a-9036-eab6b44bf994
-        5f53ce41-680f-440e-9c84-2f67c3df664d
-        6990ae39-99eb-4afa-8658-9b596915935f
-        7092d9d2-9c01-4405-8da6-ea0c423a11a1
-        8bef5068-7377-480d-9884-c7f0e0cff78d
-        974a3485-cadf-4692-9b2a-3e364015020c
-        9a7afc6d-e09f-4b8c-a525-94e8816b5798
-        9da5750a-e4e5-4071-b8ff-881c61990237
-        a601260b-b77e-4927-b463-78991dec4a56
-        c66a6166-7574-4cb3-8ea0-0580e5c215e5
-        e4fe4ae9-eea8-43c5-82f7-1dcb91a9e899
-        fb5d69b8-cd4b-443f-b63c-10e7cacf2944
-      )
-    )
-    (group "" (id a29d9d13-7df1-494a-b3a2-b0d3764b6300)
-      (members
-        2a87673a-51cd-4eb4-b2cc-f857253ed51f
-        2deed15e-a9a1-47af-80b0-81602234a3e9
-        42cfeb75-5d65-4e0b-94f8-bfdd8f57fd49
-        58a75c4a-c62e-472f-94e9-2e06d9bf6c52
-        7a8461ba-1c7a-48a4-89a1-6196ab13a810
-        81bc476a-f301-4d32-841a-7c624f900a19
-        829a8f27-f63a-419a-a25d-746295a61dd1
-        84ff41d9-332a-4b10-8bb3-6341ced16bc4
-        a0e55342-a197-4598-a137-9b40ffdc5a9f
-        a7a33e04-1f22-411a-81cf-de5556de2fe3
-        c2a71337-54dd-421c-8d71-159263d9ff28
-        c71cff5c-d4ba-4690-8f95-a3172797092b
-        d788d39c-94a2-4247-87e8-230cce608869
-        d892abb5-4f2b-4e19-9d57-6e80d27cda2f
-        dd93eabb-001c-4a67-bf26-df11a912c0cb
-        e4802904-e49e-4bef-9996-36c95d544582
+        2fe1e155-c442-4ade-a13e-00336d5adbe2
+        412a3188-9936-4aff-b746-8b6d742e0120
+        71bb735c-6c3d-4ac7-b54e-7921c8184f3d
+        77714e01-3635-4b07-9cbf-029a579e1cb5
+        9d9f2eee-beb7-45a2-b0a2-cb81d59eefb6
+        a34a3c4b-de2c-4d9f-b9a8-b40220e256d8
+        b430ce4f-826a-45f7-83e0-ad8f0a7345dd
+        cbda9a42-b908-4ff5-81e3-60a058a10548
+        f096fa3d-243e-4a71-a1a6-efb196b4b4a4
       )
     )
   )
-  (zone (net 0) (net_name "") (layer "F.Cu") (hatch edge 0.508)
-    (connect_pads (clearance 0.508))
-    (min_thickness 0.254) (filled_areas_thickness no)
-    (fill yes (thermal_gap 0.508) (thermal_bridge_width 0.508))
-    (polygon
-      (pts
-        (xy 283.3 114.8)
-        (xy 15.3 114.8)
-        (xy 15.3 78.8)
-        (xy 283.3 78.8)
+  (footprint "CIS:CIS_Edge_L1" (layer "F.Cu")
+    (at 16.62132 125)
+    (attr through_hole board_only exclude_from_pos_files exclude_from_bom)
+    (fp_text reference "REF**" (at 0.05 7 unlocked) (layer "F.SilkS") hide
+      (effects (font (size 1 1) (thickness 0.15)))
+    )
+    (fp_text value "CIS_Edge_1" (at 0 6.9 unlocked) (layer "F.Fab") hide
+      (effects (font (size 1 1) (thickness 0.15)))
+    )
+    (fp_line (start 3 0) (end 261 0) (layer "Edge.Cuts") (width 0.5))
+    (fp_line (start 264 -3) (end 264 -29) (layer "Edge.Cuts") (width 0.5))
+    (fp_line (start 261 -32) (end 3 -32) (layer "Edge.Cuts") (width 0.5))
+    (fp_line (start 0 -29) (end 0 -3) (layer "Edge.Cuts") (width 0.5))
+    (fp_arc (start 3 0) (mid 0.87868 -0.87868) (end 0 -3) (layer "Edge.Cuts") (width 0.5))
+    (fp_arc (start 264 -3) (mid 263.12132 -0.87868) (end 261 0) (layer "Edge.Cuts") (width 0.5))
+    (fp_arc (start 0 -29) (mid 0.87868 -31.12132) (end 3 -32) (layer "Edge.Cuts") (width 0.5))
+    (fp_arc (start 261 -32) (mid 263.12132 -31.12132) (end 264 -29) (layer "Edge.Cuts") (width 0.5))
+    (group "" (id 84e629d6-7948-412a-862b-6ef03beadba9)
+      (members
+        20ebd716-7865-4a7a-926b-6580938e50b8
+        445ca6aa-ab4c-41d4-acb2-e9ba5dd369b5
+        45ff495a-eca1-4e1c-8582-c39bde7122bd
+        54b9f28d-605f-4d29-83b7-6eeb198bcc53
+        5738ae7b-8832-49c6-be28-bc61572f6c95
+        728607ff-96ec-416e-98db-5d379ed06af3
+        77e79853-bc66-435f-bfda-afa20e08405e
+        cedbad8a-08bb-49ce-a1a1-a2722d67a87c
+        d52d6c78-a541-448e-abe2-26f3f88436fa
       )
     )
   )
+  (gr_rect (start 253.92132 99.85) (end 22.62132 118.15) (layer "Edge.Cuts") (width 0.5) (fill none))
 )
