File: L4/L4.kicad_pcb (KiCad board)
At the start: 2 copper layers, 264 x 32 mm, 2 parts

Commit message: Update L5 and L4 layer
Routing:
- added copper zone on B.Cu, net (none)
- added copper zone on F.Cu, net (none)
