File: LB/LB.kicad_pcb (KiCad board)
At the start: 2 copper layers, 264 x 32 mm, 4 parts

Commit message: Clean project
Parts:
- REF**: footprint CIS:CIS_Edge_Holes -> CIS:CIS_Edge_Holes_In
Changed lines of the file:
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@@
     )
   )
-  (footprint "CIS:CIS_Edge_Holes" (layer "F.Cu")
+  (footprint "CIS:CIS_Edge_Holes_In" (layer "F.Cu")
     (at 16.62132 125)
     (attr through_hole board_only exclude_from_pos_files exclude_from_bom)
@@
         (effects (font (size 1 1) (thickness 0.15)))
     )
-    (pad "" thru_hole circle (at 3.5 -28.5) (size 3 3) (drill 2.2) (layers "*.Cu" "*.Mask"))
-    (pad "" thru_hole circle (at 3.5 -3.5) (size 3 3) (drill 2.2) (layers "*.Cu" "*.Mask"))
-    (pad "" thru_hole circle (at 88 -28.5) (size 3 3) (drill 2.2) (layers "*.Cu" "*.Mask"))
-    (pad "" thru_hole circle (at 88 -3.5) (size 3 3) (drill 2.2) (layers "*.Cu" "*.Mask"))
-    (pad "" thru_hole circle (at 176 -28.5) (size 3 3) (drill 2.2) (layers "*.Cu" "*.Mask"))
-    (pad "" thru_hole circle (at 176 -3.5287) (size 3 3) (drill 2.2) (layers "*.Cu" "*.Mask"))
-    (pad "" thru_hole circle (at 260.5 -28.5) (size 3 3) (drill 2.2) (layers "*.Cu" "*.Mask"))
-    (pad "" thru_hole circle (at 260.5 -3.5) (size 3 3) (drill 2.2) (layers "*.Cu" "*.Mask"))
-    (group "" (id 42a9493b-299e-433f-8afb-aba2ca5a0459)
+    (pad "" thru_hole circle (at 3.5 -28.5) (size 4 4) (drill 3.1) (layers "*.Cu" "*.Mask"))
+    (pad "" thru_hole circle (at 3.5 -3.5) (size 4 4) (drill 3.1) (layers "*.Cu" "*.Mask"))
+    (pad "" thru_hole circle (at 88 -28.5) (size 4 4) (drill 3.1) (layers "*.Cu" "*.Mask"))
+    (pad "" thru_hole circle (at 88 -3.5) (size 4 4) (drill 3.1) (layers "*.Cu" "*.Mask"))
+    (pad "" thru_hole circle (at 176 -28.5) (size 4 4) (drill 3.1) (layers "*.Cu" "*.Mask"))
+    (pad "" thru_hole circle (at 176 -3.5287) (size 4 4) (drill 3.1) (layers "*.Cu" "*.Mask"))
+    (pad "" thru_hole circle (at 260.5 -28.5) (size 4 4) (drill 3.1) (layers "*.Cu" "*.Mask"))
+    (pad "" thru_hole circle (at 260.5 -3.5) (size 4 4) (drill 3.1) (layers "*.Cu" "*.Mask"))
+    (group "" (id 06c4bb1d-989a-41e3-b52e-45917ab24997)
       (members
-        3dd08fce-ac7d-49a9-94f3-e2ba54f29902
-        6768afe3-01c8-4606-a632-654a1521139a
-        7e332f99-da6d-49b6-afd0-971d6081873c
-        be23ae56-261a-4ed7-ad31-2f816396d6c7
-        e70d3230-a2bb-4eb3-9efa-291ab3255139
-        f0db2dba-d276-425e-af0e-022eff0ea206
-        f5f3b307-d647-4e03-9e31-f12b7b83f5fd
-        f65d9575-1c26-4a51-a4c7-0b419b680a4f
-        f841a204-2a95-4897-a638-5a69ffe2c024
+        2403b100-8eb3-4f40-9b20-ce71fb90940d
+        2c4b7ad0-cc08-44a1-a9a5-16f6ac99a634
+        349ae92a-c492-4034-a268-dcc498797ef6
+        645a8216-3f41-42d8-bb06-84492e228e35
+        7702d058-639d-4e3d-9bff-d15eb0697b8c
+        80295565-0ccc-4044-a2c5-694a22489195
+        83e2f7a9-dd24-4961-ae78-27e4705e8da3
+        a5c36d8f-bd0a-42ca-a588-cc2ef8509644
+        b769ab35-21c1-408d-9a42-8a3d9fa231a7
       )
     )
@@
     (pts (xy 258.52132 117.45) (xy 258.52132 118.15))
     (height -3.599999)
-    (gr_text "0,7 mm" (at 260.971319 117.8 90) (layer "F.Fab")
+    (gr_text "0.7 mm" (at 260.971319 117.8 90) (layer "F.Fab")
       (effects (font (size 1 1) (thickness 0.15)))
     )
@@
     (pts (xy 253.92132 118.15) (xy 22.62132 118.15))
     (height -2.85)
-    (gr_text "231,3 mm" (at 138.27132 119.85) (layer "F.Fab")
+    (gr_text "231.3 mm" (at 138.27132 119.85) (layer "F.Fab")
       (effects (font (size 1 1) (thickness 0.15)))
     )
@@
     (pts (xy 22.62132 118.15) (xy 22.62132 99.85))
     (height -2.5)
-    (gr_text "18,3 mm" (at 18.97132 109 90) (layer "F.Fab")
+    (gr_text "18.3 mm" (at 18.97132 109 90) (layer "F.Fab")
       (effects (font (size 1 1) (thickness 0.15)))
     )
@@
     (pts (xy 258.52132 117.45) (xy 258.52132 100.55))
     (height -1.5)
-    (gr_text "16,9 mm" (at 255.87132 109 90) (layer "F.Fab")
+    (gr_text "16.9 mm" (at 255.87132 109 90) (layer "F.Fab")
       (effects (font (size 1 1) (thickness 0.15)))
     )

Commit message: Update holes
Changed lines of the file:
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@@
         (effects (font (size 1 1) (thickness 0.15)))
     )
-    (pad "" thru_hole circle (at 3.5 -28.5) (size 4 4) (drill 3.1) (layers "*.Cu" "*.Mask"))
-    (pad "" thru_hole circle (at 3.5 -3.5) (size 4 4) (drill 3.1) (layers "*.Cu" "*.Mask"))
-    (pad "" thru_hole circle (at 88 -28.5) (size 4 4) (drill 3.1) (layers "*.Cu" "*.Mask"))
-    (pad "" thru_hole circle (at 88 -3.5) (size 4 4) (drill 3.1) (layers "*.Cu" "*.Mask"))
-    (pad "" thru_hole circle (at 176 -28.5) (size 4 4) (drill 3.1) (layers "*.Cu" "*.Mask"))
-    (pad "" thru_hole circle (at 176 -3.5287) (size 4 4) (drill 3.1) (layers "*.Cu" "*.Mask"))
-    (pad "" thru_hole circle (at 260.5 -28.5) (size 4 4) (drill 3.1) (layers "*.Cu" "*.Mask"))
-    (pad "" thru_hole circle (at 260.5 -3.5) (size 4 4) (drill 3.1) (layers "*.Cu" "*.Mask"))
-    (group "" (id 06c4bb1d-989a-41e3-b52e-45917ab24997)
+    (pad "" thru_hole circle (at 3.5 -28.5) (size 4 4) (drill 3.2) (layers "*.Cu" "*.Mask"))
+    (pad "" thru_hole circle (at 3.5 -3.5) (size 4 4) (drill 3.2) (layers "*.Cu" "*.Mask"))
+    (pad "" thru_hole circle (at 88 -28.5) (size 4 4) (drill 3.2) (layers "*.Cu" "*.Mask"))
+    (pad "" thru_hole circle (at 88 -3.5) (size 4 4) (drill 3.2) (layers "*.Cu" "*.Mask"))
+    (pad "" thru_hole circle (at 176 -28.5) (size 4 4) (drill 3.2) (layers "*.Cu" "*.Mask"))
+    (pad "" thru_hole circle (at 176 -3.5287) (size 4 4) (drill 3.2) (layers "*.Cu" "*.Mask"))
+    (pad "" thru_hole circle (at 260.5 -28.5) (size 4 4) (drill 3.2) (layers "*.Cu" "*.Mask"))
+    (pad "" thru_hole circle (at 260.5 -3.5) (size 4 4) (drill 3.2) (layers "*.Cu" "*.Mask"))
+    (group "" (id 4ae57018-3b8b-46c9-a187-dc479517b62d)
       (members
-        2403b100-8eb3-4f40-9b20-ce71fb90940d
-        2c4b7ad0-cc08-44a1-a9a5-16f6ac99a634
-        349ae92a-c492-4034-a268-dcc498797ef6
-        645a8216-3f41-42d8-bb06-84492e228e35
-        7702d058-639d-4e3d-9bff-d15eb0697b8c
-        80295565-0ccc-4044-a2c5-694a22489195
-        83e2f7a9-dd24-4961-ae78-27e4705e8da3
-        a5c36d8f-bd0a-42ca-a588-cc2ef8509644
-        b769ab35-21c1-408d-9a42-8a3d9fa231a7
+        0863a3f5-9cfb-4462-b6aa-d0e69bf7c11d
+        0a26b8f4-5eb5-48d8-ae96-27c77be7b662
+        3135c2e9-7925-47f2-b244-ea2efe5d2531
+        462290d8-7e21-4e4b-bc05-8b41d3a26cd6
+        986def10-311a-4e79-a608-32610947dd2d
+        bb1556e4-2f4c-4e30-991e-80d103472dc3
+        bb532749-8dab-4cbd-8899-96b115fb9b87
+        c8b00072-dd9b-4ec9-ab8f-bf0809be9e39
+        e93df73d-f169-46d1-9371-183c1ea2d669
       )
     )
