File: LC/LC.kicad_pcb (KiCad board)
At the start: 2 copper layers, 264 x 32 mm, 2 parts

Commit message: Clean project
Parts:
- REF**: footprint CIS:CIS_Edge_Holes -> CIS:CIS_Edge_Holes_In
Changed lines of the file:
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@@
     )
   )
-  (footprint "CIS:CIS_Edge_Holes" (layer "F.Cu")
+  (footprint "CIS:CIS_Edge_Holes_In" (layer "F.Cu")
     (at 16.62132 125)
     (attr through_hole board_only exclude_from_pos_files exclude_from_bom)
@@
         (effects (font (size 1 1) (thickness 0.15)))
     )
-    (pad "" thru_hole circle (at 3.5 -28.5) (size 3 3) (drill 2.2) (layers "*.Cu" "*.Mask"))
-    (pad "" thru_hole circle (at 3.5 -3.5) (size 3 3) (drill 2.2) (layers "*.Cu" "*.Mask"))
-    (pad "" thru_hole circle (at 88 -28.5) (size 3 3) (drill 2.2) (layers "*.Cu" "*.Mask"))
-    (pad "" thru_hole circle (at 88 -3.5) (size 3 3) (drill 2.2) (layers "*.Cu" "*.Mask"))
-    (pad "" thru_hole circle (at 176 -28.5) (size 3 3) (drill 2.2) (layers "*.Cu" "*.Mask"))
-    (pad "" thru_hole circle (at 176 -3.5287) (size 3 3) (drill 2.2) (layers "*.Cu" "*.Mask"))
-    (pad "" thru_hole circle (at 260.5 -28.5) (size 3 3) (drill 2.2) (layers "*.Cu" "*.Mask"))
-    (pad "" thru_hole circle (at 260.5 -3.5) (size 3 3) (drill 2.2) (layers "*.Cu" "*.Mask"))
-    (group "" (id 42a9493b-299e-433f-8afb-aba2ca5a0459)
+    (pad "" thru_hole circle (at 3.5 -28.5) (size 4 4) (drill 3.1) (layers "*.Cu" "*.Mask"))
+    (pad "" thru_hole circle (at 3.5 -3.5) (size 4 4) (drill 3.1) (layers "*.Cu" "*.Mask"))
+    (pad "" thru_hole circle (at 88 -28.5) (size 4 4) (drill 3.1) (layers "*.Cu" "*.Mask"))
+    (pad "" thru_hole circle (at 88 -3.5) (size 4 4) (drill 3.1) (layers "*.Cu" "*.Mask"))
+    (pad "" thru_hole circle (at 176 -28.5) (size 4 4) (drill 3.1) (layers "*.Cu" "*.Mask"))
+    (pad "" thru_hole circle (at 176 -3.5287) (size 4 4) (drill 3.1) (layers "*.Cu" "*.Mask"))
+    (pad "" thru_hole circle (at 260.5 -28.5) (size 4 4) (drill 3.1) (layers "*.Cu" "*.Mask"))
+    (pad "" thru_hole circle (at 260.5 -3.5) (size 4 4) (drill 3.1) (layers "*.Cu" "*.Mask"))
+    (group "" (id 0cb43c7f-7c82-4eba-a58c-810e33488cd4)
       (members
-        3dd08fce-ac7d-49a9-94f3-e2ba54f29902
-        6768afe3-01c8-4606-a632-654a1521139a
-        7e332f99-da6d-49b6-afd0-971d6081873c
-        be23ae56-261a-4ed7-ad31-2f816396d6c7
-        e70d3230-a2bb-4eb3-9efa-291ab3255139
-        f0db2dba-d276-425e-af0e-022eff0ea206
-        f5f3b307-d647-4e03-9e31-f12b7b83f5fd
-        f65d9575-1c26-4a51-a4c7-0b419b680a4f
-        f841a204-2a95-4897-a638-5a69ffe2c024
+        0f99f63b-cb22-4b1e-a92d-21e5368fab6e
+        1c7776cb-03fc-4d27-860a-6a915f863990
+        3e8ff678-1bbf-4500-937a-864e41eb36a4
+        579c2a38-5925-4bd1-9296-c2edb7fb9513
+        5a26e2cc-6956-447b-b410-f5a7b8221886
+        6ad70569-8298-4730-98fd-9a4937fbcb88
+        a88f6740-38a9-4b78-8bdb-ef8241f9cc00
+        b808cc1f-c6bf-4168-a992-9a6052e3d066
+        ea4bd7e4-70e7-426f-a88f-9a7b5106d0bd
       )
     )
@@
     (pts (xy 258.52132 117.45) (xy 258.52132 118.15))
     (height -3.599999)
-    (gr_text "0,7 mm" (at 260.971319 117.8 90) (layer "F.Fab")
+    (gr_text "0.7 mm" (at 260.971319 117.8 90) (layer "F.Fab")
       (effects (font (size 1 1) (thickness 0.15)))
     )
@@
     (pts (xy 16.62132 101.75) (xy 36.12132 101.75))
     (height -11.25)
-    (gr_text "19,5 mm" (at 26.37132 89.35) (layer "F.Fab")
+    (gr_text "19.5 mm" (at 26.37132 89.35) (layer "F.Fab")
       (effects (font (size 1 1) (thickness 0.15)))
     )
@@
     (pts (xy 36.12132 101.75) (xy 55.12132 101.75))
     (height -11.25)
-    (gr_text "19,0000 mm" (at 45.62132 89.35) (layer "F.Fab")
+    (gr_text "19.0000 mm" (at 45.62132 89.35) (layer "F.Fab")
       (effects (font (size 1 1) (thickness 0.15)))
     )

Commit message: Update holes
Changed lines of the file:
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@@
         (effects (font (size 1 1) (thickness 0.15)))
     )
-    (pad "" thru_hole circle (at 3.5 -28.5) (size 4 4) (drill 3.1) (layers "*.Cu" "*.Mask"))
-    (pad "" thru_hole circle (at 3.5 -3.5) (size 4 4) (drill 3.1) (layers "*.Cu" "*.Mask"))
-    (pad "" thru_hole circle (at 88 -28.5) (size 4 4) (drill 3.1) (layers "*.Cu" "*.Mask"))
-    (pad "" thru_hole circle (at 88 -3.5) (size 4 4) (drill 3.1) (layers "*.Cu" "*.Mask"))
-    (pad "" thru_hole circle (at 176 -28.5) (size 4 4) (drill 3.1) (layers "*.Cu" "*.Mask"))
-    (pad "" thru_hole circle (at 176 -3.5287) (size 4 4) (drill 3.1) (layers "*.Cu" "*.Mask"))
-    (pad "" thru_hole circle (at 260.5 -28.5) (size 4 4) (drill 3.1) (layers "*.Cu" "*.Mask"))
-    (pad "" thru_hole circle (at 260.5 -3.5) (size 4 4) (drill 3.1) (layers "*.Cu" "*.Mask"))
-    (group "" (id 0cb43c7f-7c82-4eba-a58c-810e33488cd4)
+    (pad "" thru_hole circle (at 3.5 -28.5) (size 4 4) (drill 3.2) (layers "*.Cu" "*.Mask"))
+    (pad "" thru_hole circle (at 3.5 -3.5) (size 4 4) (drill 3.2) (layers "*.Cu" "*.Mask"))
+    (pad "" thru_hole circle (at 88 -28.5) (size 4 4) (drill 3.2) (layers "*.Cu" "*.Mask"))
+    (pad "" thru_hole circle (at 88 -3.5) (size 4 4) (drill 3.2) (layers "*.Cu" "*.Mask"))
+    (pad "" thru_hole circle (at 176 -28.5) (size 4 4) (drill 3.2) (layers "*.Cu" "*.Mask"))
+    (pad "" thru_hole circle (at 176 -3.5287) (size 4 4) (drill 3.2) (layers "*.Cu" "*.Mask"))
+    (pad "" thru_hole circle (at 260.5 -28.5) (size 4 4) (drill 3.2) (layers "*.Cu" "*.Mask"))
+    (pad "" thru_hole circle (at 260.5 -3.5) (size 4 4) (drill 3.2) (layers "*.Cu" "*.Mask"))
+    (group "" (id d6ac9ea1-c190-4a67-878c-4e6617bcc114)
       (members
-        0f99f63b-cb22-4b1e-a92d-21e5368fab6e
-        1c7776cb-03fc-4d27-860a-6a915f863990
-        3e8ff678-1bbf-4500-937a-864e41eb36a4
-        579c2a38-5925-4bd1-9296-c2edb7fb9513
-        5a26e2cc-6956-447b-b410-f5a7b8221886
-        6ad70569-8298-4730-98fd-9a4937fbcb88
-        a88f6740-38a9-4b78-8bdb-ef8241f9cc00
-        b808cc1f-c6bf-4168-a992-9a6052e3d066
-        ea4bd7e4-70e7-426f-a88f-9a7b5106d0bd
+        01ee91b5-660d-44c2-9ce7-ba9468ed43f9
+        351fa8bc-c4c3-49ab-8581-693dfbb7cfef
+        5d2216b2-d2dd-4db9-994b-1fc6c9599b94
+        8fb427a1-fc1e-494f-9d51-78c01dd60fbf
+        9acfbd4b-4c1c-4797-b077-0fa9b0e8be24
+        9f568243-4f76-41aa-a9ca-651c27247192
+        ad2df375-07fa-4dcd-83d9-680f75eee3c7
+        bc6fcfc1-01a2-4135-9e6a-aba28a6fff14
+        f7ac481c-737f-491f-9061-56fc9b737da1
       )
     )
@@
     (pts (xy 258.52132 117.45) (xy 258.52132 118.15))
     (height -3.599999)
-    (gr_text "0.7 mm" (at 260.971319 117.8 90) (layer "F.Fab")
+    (gr_text "0,7 mm" (at 260.971319 117.8 90) (layer "F.Fab")
       (effects (font (size 1 1) (thickness 0.15)))
     )
@@
     (pts (xy 16.62132 101.75) (xy 36.12132 101.75))
     (height -11.25)
-    (gr_text "19.5 mm" (at 26.37132 89.35) (layer "F.Fab")
+    (gr_text "19,5 mm" (at 26.37132 89.35) (layer "F.Fab")
       (effects (font (size 1 1) (thickness 0.15)))
     )
@@
     (pts (xy 36.12132 101.75) (xy 55.12132 101.75))
     (height -11.25)
-    (gr_text "19.0000 mm" (at 45.62132 89.35) (layer "F.Fab")
+    (gr_text "19,0000 mm" (at 45.62132 89.35) (layer "F.Fab")
       (effects (font (size 1 1) (thickness 0.15)))
     )
