File: LD/LD.kicad_pcb (KiCad board)
At the start: 2 copper layers, 264 x 32 mm, 2 parts

Commit message: Clean project
Parts:
- REF**: footprint CIS:CIS_Edge_Holes -> CIS:CIS_Edge_Holes_In
Changed lines of the file:
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@@
     )
   )
-  (footprint "CIS:CIS_Edge_Holes" (layer "F.Cu")
+  (footprint "CIS:CIS_Edge_Holes_In" (layer "F.Cu")
     (at 16.62132 125)
     (attr through_hole board_only exclude_from_pos_files exclude_from_bom)
@@
         (effects (font (size 1 1) (thickness 0.15)))
     )
-    (pad "" thru_hole circle (at 3.5 -28.5) (size 3 3) (drill 2.2) (layers "*.Cu" "*.Mask"))
-    (pad "" thru_hole circle (at 3.5 -3.5) (size 3 3) (drill 2.2) (layers "*.Cu" "*.Mask"))
-    (pad "" thru_hole circle (at 88 -28.5) (size 3 3) (drill 2.2) (layers "*.Cu" "*.Mask"))
-    (pad "" thru_hole circle (at 88 -3.5) (size 3 3) (drill 2.2) (layers "*.Cu" "*.Mask"))
-    (pad "" thru_hole circle (at 176 -28.5) (size 3 3) (drill 2.2) (layers "*.Cu" "*.Mask"))
-    (pad "" thru_hole circle (at 176 -3.5287) (size 3 3) (drill 2.2) (layers "*.Cu" "*.Mask"))
-    (pad "" thru_hole circle (at 260.5 -28.5) (size 3 3) (drill 2.2) (layers "*.Cu" "*.Mask"))
-    (pad "" thru_hole circle (at 260.5 -3.5) (size 3 3) (drill 2.2) (layers "*.Cu" "*.Mask"))
-    (group "" (id 42a9493b-299e-433f-8afb-aba2ca5a0459)
+    (pad "" thru_hole circle (at 3.5 -28.5) (size 4 4) (drill 3.1) (layers "*.Cu" "*.Mask"))
+    (pad "" thru_hole circle (at 3.5 -3.5) (size 4 4) (drill 3.1) (layers "*.Cu" "*.Mask"))
+    (pad "" thru_hole circle (at 88 -28.5) (size 4 4) (drill 3.1) (layers "*.Cu" "*.Mask"))
+    (pad "" thru_hole circle (at 88 -3.5) (size 4 4) (drill 3.1) (layers "*.Cu" "*.Mask"))
+    (pad "" thru_hole circle (at 176 -28.5) (size 4 4) (drill 3.1) (layers "*.Cu" "*.Mask"))
+    (pad "" thru_hole circle (at 176 -3.5287) (size 4 4) (drill 3.1) (layers "*.Cu" "*.Mask"))
+    (pad "" thru_hole circle (at 260.5 -28.5) (size 4 4) (drill 3.1) (layers "*.Cu" "*.Mask"))
+    (pad "" thru_hole circle (at 260.5 -3.5) (size 4 4) (drill 3.1) (layers "*.Cu" "*.Mask"))
+    (group "" (id 188fa7e0-f617-4383-b94e-900c0ea992bf)
       (members
-        3dd08fce-ac7d-49a9-94f3-e2ba54f29902
-        6768afe3-01c8-4606-a632-654a1521139a
-        7e332f99-da6d-49b6-afd0-971d6081873c
-        be23ae56-261a-4ed7-ad31-2f816396d6c7
-        e70d3230-a2bb-4eb3-9efa-291ab3255139
-        f0db2dba-d276-425e-af0e-022eff0ea206
-        f5f3b307-d647-4e03-9e31-f12b7b83f5fd
-        f65d9575-1c26-4a51-a4c7-0b419b680a4f
-        f841a204-2a95-4897-a638-5a69ffe2c024
+        46d6c7ea-6705-48f9-96b9-209f581747ed
+        7a7d51fa-8f2a-4346-b430-27803aea5ebe
+        a21044b3-c931-494e-afb1-61d15fc9f9dd
+        a38c6cdb-e940-4e96-b77c-66a21214a1e4
+        a93a93de-9ba1-4724-9a31-e93e87d0d0ec
+        b0f62e96-c0cb-4e98-bf1b-b72c708f6fd6
+        f44c1191-0da3-4839-b70a-505a84a3a38a
+        f6eb3e91-3289-4d1c-9079-2ad917558508
+        fd5ec640-8fbb-411c-9a9c-3dcffa0ab375
       )
     )
@@
     (pts (xy 258.52132 117.45) (xy 258.52132 118.15))
     (height -3.599999)
-    (gr_text "0,7 mm" (at 260.971319 117.8 90) (layer "F.Fab")
+    (gr_text "0.7 mm" (at 260.971319 117.8 90) (layer "F.Fab")
       (effects (font (size 1 1) (thickness 0.15)))
     )
@@
     (pts (xy 253.92132 118.15) (xy 22.62132 118.15))
     (height -5.35)
-    (gr_text "231,3 mm" (at 138.27132 122.35) (layer "F.Fab")
+    (gr_text "231.3 mm" (at 138.27132 122.35) (layer "F.Fab")
       (effects (font (size 1 1) (thickness 0.15)))
     )
@@
     (pts (xy 258.52132 117.45) (xy 258.52132 100.55))
     (height -1.5)
-    (gr_text "16,9 mm" (at 255.87132 109 90) (layer "F.Fab")
+    (gr_text "16.9 mm" (at 255.87132 109 90) (layer "F.Fab")
       (effects (font (size 1 1) (thickness 0.15)))
     )
@@
     (pts (xy 22.62132 121) (xy 22.62132 97))
     (height -7.5)
-    (gr_text "24,0000 mm" (at 13.97132 109 90) (layer "F.Fab")
+    (gr_text "24.0000 mm" (at 13.97132 109 90) (layer "F.Fab")
       (effects (font (size 1 1) (thickness 0.15)))
     )

Commit message: Update holes
Changed lines of the file:
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@@
         (effects (font (size 1 1) (thickness 0.15)))
     )
-    (pad "" thru_hole circle (at 3.5 -28.5) (size 4 4) (drill 3.1) (layers "*.Cu" "*.Mask"))
-    (pad "" thru_hole circle (at 3.5 -3.5) (size 4 4) (drill 3.1) (layers "*.Cu" "*.Mask"))
-    (pad "" thru_hole circle (at 88 -28.5) (size 4 4) (drill 3.1) (layers "*.Cu" "*.Mask"))
-    (pad "" thru_hole circle (at 88 -3.5) (size 4 4) (drill 3.1) (layers "*.Cu" "*.Mask"))
-    (pad "" thru_hole circle (at 176 -28.5) (size 4 4) (drill 3.1) (layers "*.Cu" "*.Mask"))
-    (pad "" thru_hole circle (at 176 -3.5287) (size 4 4) (drill 3.1) (layers "*.Cu" "*.Mask"))
-    (pad "" thru_hole circle (at 260.5 -28.5) (size 4 4) (drill 3.1) (layers "*.Cu" "*.Mask"))
-    (pad "" thru_hole circle (at 260.5 -3.5) (size 4 4) (drill 3.1) (layers "*.Cu" "*.Mask"))
-    (group "" (id 188fa7e0-f617-4383-b94e-900c0ea992bf)
+    (pad "" thru_hole circle (at 3.5 -28.5) (size 4 4) (drill 3.2) (layers "*.Cu" "*.Mask"))
+    (pad "" thru_hole circle (at 3.5 -3.5) (size 4 4) (drill 3.2) (layers "*.Cu" "*.Mask"))
+    (pad "" thru_hole circle (at 88 -28.5) (size 4 4) (drill 3.2) (layers "*.Cu" "*.Mask"))
+    (pad "" thru_hole circle (at 88 -3.5) (size 4 4) (drill 3.2) (layers "*.Cu" "*.Mask"))
+    (pad "" thru_hole circle (at 176 -28.5) (size 4 4) (drill 3.2) (layers "*.Cu" "*.Mask"))
+    (pad "" thru_hole circle (at 176 -3.5287) (size 4 4) (drill 3.2) (layers "*.Cu" "*.Mask"))
+    (pad "" thru_hole circle (at 260.5 -28.5) (size 4 4) (drill 3.2) (layers "*.Cu" "*.Mask"))
+    (pad "" thru_hole circle (at 260.5 -3.5) (size 4 4) (drill 3.2) (layers "*.Cu" "*.Mask"))
+    (group "" (id 759a0691-3c47-484b-a1cb-5ddb1ebbbdb7)
       (members
-        46d6c7ea-6705-48f9-96b9-209f581747ed
-        7a7d51fa-8f2a-4346-b430-27803aea5ebe
-        a21044b3-c931-494e-afb1-61d15fc9f9dd
-        a38c6cdb-e940-4e96-b77c-66a21214a1e4
-        a93a93de-9ba1-4724-9a31-e93e87d0d0ec
-        b0f62e96-c0cb-4e98-bf1b-b72c708f6fd6
-        f44c1191-0da3-4839-b70a-505a84a3a38a
-        f6eb3e91-3289-4d1c-9079-2ad917558508
-        fd5ec640-8fbb-411c-9a9c-3dcffa0ab375
+        07e47ca5-ff22-4843-8ede-59ea7a7cde5d
+        13401ab6-275a-412a-bc87-7c2efa937d2d
+        1cc7f942-7aeb-4993-81f6-121179ba1554
+        4848d874-72f5-47a2-b8ed-3260bcd881cd
+        56c2da0e-0ef4-4cb2-a530-7f590160e3f3
+        762239b9-d70a-4a39-8c2b-2e4ac3490a1d
+        ad901ce7-74a9-443a-8a36-be7d99738122
+        c7e5a777-5a0b-4136-b86f-96bfbdb6d031
+        f076c320-fcbd-4123-a5bd-485b47b3cf01
       )
     )
