File: LE/LE.kicad_pcb (KiCad board)
At the start: 2 copper layers, 264 x 32 mm, 2 parts

Commit message: Clean project
Parts:
- REF**: footprint CIS:CIS_Edge_Holes -> CIS:CIS_Edge_Holes_In
Changed lines of the file:
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@@
     )
   )
-  (footprint "CIS:CIS_Edge_Holes" (layer "F.Cu")
+  (footprint "CIS:CIS_Edge_Holes_In" (layer "F.Cu")
     (at 16.62132 125)
     (attr through_hole board_only exclude_from_pos_files exclude_from_bom)
@@
         (effects (font (size 1 1) (thickness 0.15)))
     )
-    (pad "" thru_hole circle (at 3.5 -28.5) (size 3 3) (drill 2.2) (layers "*.Cu" "*.Mask"))
-    (pad "" thru_hole circle (at 3.5 -3.5) (size 3 3) (drill 2.2) (layers "*.Cu" "*.Mask"))
-    (pad "" thru_hole circle (at 88 -28.5) (size 3 3) (drill 2.2) (layers "*.Cu" "*.Mask"))
-    (pad "" thru_hole circle (at 88 -3.5) (size 3 3) (drill 2.2) (layers "*.Cu" "*.Mask"))
-    (pad "" thru_hole circle (at 176 -28.5) (size 3 3) (drill 2.2) (layers "*.Cu" "*.Mask"))
-    (pad "" thru_hole circle (at 176 -3.5287) (size 3 3) (drill 2.2) (layers "*.Cu" "*.Mask"))
-    (pad "" thru_hole circle (at 260.5 -28.5) (size 3 3) (drill 2.2) (layers "*.Cu" "*.Mask"))
-    (pad "" thru_hole circle (at 260.5 -3.5) (size 3 3) (drill 2.2) (layers "*.Cu" "*.Mask"))
-    (group "" (id 42a9493b-299e-433f-8afb-aba2ca5a0459)
+    (pad "" thru_hole circle (at 3.5 -28.5) (size 4 4) (drill 3.1) (layers "*.Cu" "*.Mask"))
+    (pad "" thru_hole circle (at 3.5 -3.5) (size 4 4) (drill 3.1) (layers "*.Cu" "*.Mask"))
+    (pad "" thru_hole circle (at 88 -28.5) (size 4 4) (drill 3.1) (layers "*.Cu" "*.Mask"))
+    (pad "" thru_hole circle (at 88 -3.5) (size 4 4) (drill 3.1) (layers "*.Cu" "*.Mask"))
+    (pad "" thru_hole circle (at 176 -28.5) (size 4 4) (drill 3.1) (layers "*.Cu" "*.Mask"))
+    (pad "" thru_hole circle (at 176 -3.5287) (size 4 4) (drill 3.1) (layers "*.Cu" "*.Mask"))
+    (pad "" thru_hole circle (at 260.5 -28.5) (size 4 4) (drill 3.1) (layers "*.Cu" "*.Mask"))
+    (pad "" thru_hole circle (at 260.5 -3.5) (size 4 4) (drill 3.1) (layers "*.Cu" "*.Mask"))
+    (group "" (id f026bee6-e341-493a-8e05-498d51c37ff7)
       (members
-        3dd08fce-ac7d-49a9-94f3-e2ba54f29902
-        6768afe3-01c8-4606-a632-654a1521139a
-        7e332f99-da6d-49b6-afd0-971d6081873c
-        be23ae56-261a-4ed7-ad31-2f816396d6c7
-        e70d3230-a2bb-4eb3-9efa-291ab3255139
-        f0db2dba-d276-425e-af0e-022eff0ea206
-        f5f3b307-d647-4e03-9e31-f12b7b83f5fd
-        f65d9575-1c26-4a51-a4c7-0b419b680a4f
-        f841a204-2a95-4897-a638-5a69ffe2c024
+        072e3fe3-be39-4dc5-9341-5d388a3bcfa6
+        15ac6dea-de96-4c83-86b2-a5aa945f94f3
+        2a5ab279-6119-4535-b614-5c2085d3415c
+        363f02f9-a99b-4c5f-9247-05ad7a564fbc
+        695e7eb0-6398-4736-aa68-8d0155ebaa6c
+        6e9e07ef-601c-40eb-a287-33ee46a5786b
+        c0f62a04-fd85-4ba7-9da8-680142065562
+        d7b68d6c-bb79-4c83-b718-d216c6e93c35
+        f07ee87c-fb6b-41a4-ae19-5f9a4ccc02a0
       )
     )
@@
     (pts (xy 280.62132 96) (xy 277.92132 96))
     (height 5.2)
-    (gr_text "2,7000 mm" (at 279.27132 89.65) (layer "Edge.Cuts")
+    (gr_text "2.7000 mm" (at 279.27132 89.65) (layer "Edge.Cuts")
       (effects (font (size 1 1) (thickness 0.15)))
     )
@@
     (pts (xy 274.62132 118.15) (xy 274.62132 99.85))
     (height 2.3)
-    (gr_text "18,3 mm" (at 275.77132 109 90) (layer "F.Fab")
+    (gr_text "18.3 mm" (at 275.77132 109 90) (layer "F.Fab")
       (effects (font (size 1 1) (thickness 0.15)))
     )
@@
     (pts (xy 16.62132 113.7) (xy 19.32132 113.7))
     (height -0.8)
-    (gr_text "2,7 mm" (at 17.97132 111.75) (layer "F.Fab")
+    (gr_text "2.7 mm" (at 17.97132 111.75) (layer "F.Fab")
       (effects (font (size 1 1) (thickness 0.15)))
     )
@@
     (pts (xy 253.92132 118.15) (xy 22.62132 118.15))
     (height -5.35)
-    (gr_text "231,3 mm" (at 138.27132 122.35) (layer "F.Fab")
+    (gr_text "231.3 mm" (at 138.27132 122.35) (layer "F.Fab")
       (effects (font (size 1 1) (thickness 0.15)))
     )
@@
     (pts (xy 253.92132 96.25) (xy 253.92132 121.75))
     (height -2.7)
-    (gr_text "25,5 mm" (at 255.47132 109 90) (layer "F.Fab")
+    (gr_text "25.5 mm" (at 255.47132 109 90) (layer "F.Fab")
       (effects (font (size 1 1) (thickness 0.15)))
     )

Commit message: Update holes
Changed lines of the file:
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@@
         (effects (font (size 1 1) (thickness 0.15)))
     )
-    (pad "" thru_hole circle (at 3.5 -28.5) (size 4 4) (drill 3.1) (layers "*.Cu" "*.Mask"))
-    (pad "" thru_hole circle (at 3.5 -3.5) (size 4 4) (drill 3.1) (layers "*.Cu" "*.Mask"))
-    (pad "" thru_hole circle (at 88 -28.5) (size 4 4) (drill 3.1) (layers "*.Cu" "*.Mask"))
-    (pad "" thru_hole circle (at 88 -3.5) (size 4 4) (drill 3.1) (layers "*.Cu" "*.Mask"))
-    (pad "" thru_hole circle (at 176 -28.5) (size 4 4) (drill 3.1) (layers "*.Cu" "*.Mask"))
-    (pad "" thru_hole circle (at 176 -3.5287) (size 4 4) (drill 3.1) (layers "*.Cu" "*.Mask"))
-    (pad "" thru_hole circle (at 260.5 -28.5) (size 4 4) (drill 3.1) (layers "*.Cu" "*.Mask"))
-    (pad "" thru_hole circle (at 260.5 -3.5) (size 4 4) (drill 3.1) (layers "*.Cu" "*.Mask"))
-    (group "" (id f026bee6-e341-493a-8e05-498d51c37ff7)
+    (pad "" thru_hole circle (at 3.5 -28.5) (size 4 4) (drill 3.2) (layers "*.Cu" "*.Mask"))
+    (pad "" thru_hole circle (at 3.5 -3.5) (size 4 4) (drill 3.2) (layers "*.Cu" "*.Mask"))
+    (pad "" thru_hole circle (at 88 -28.5) (size 4 4) (drill 3.2) (layers "*.Cu" "*.Mask"))
+    (pad "" thru_hole circle (at 88 -3.5) (size 4 4) (drill 3.2) (layers "*.Cu" "*.Mask"))
+    (pad "" thru_hole circle (at 176 -28.5) (size 4 4) (drill 3.2) (layers "*.Cu" "*.Mask"))
+    (pad "" thru_hole circle (at 176 -3.5287) (size 4 4) (drill 3.2) (layers "*.Cu" "*.Mask"))
+    (pad "" thru_hole circle (at 260.5 -28.5) (size 4 4) (drill 3.2) (layers "*.Cu" "*.Mask"))
+    (pad "" thru_hole circle (at 260.5 -3.5) (size 4 4) (drill 3.2) (layers "*.Cu" "*.Mask"))
+    (group "" (id 3ed139ae-442e-4d55-86ff-e9c30492a662)
       (members
-        072e3fe3-be39-4dc5-9341-5d388a3bcfa6
-        15ac6dea-de96-4c83-86b2-a5aa945f94f3
-        2a5ab279-6119-4535-b614-5c2085d3415c
-        363f02f9-a99b-4c5f-9247-05ad7a564fbc
-        695e7eb0-6398-4736-aa68-8d0155ebaa6c
-        6e9e07ef-601c-40eb-a287-33ee46a5786b
-        c0f62a04-fd85-4ba7-9da8-680142065562
-        d7b68d6c-bb79-4c83-b718-d216c6e93c35
-        f07ee87c-fb6b-41a4-ae19-5f9a4ccc02a0
+        0625d69b-4917-41a3-83b5-9b978d86ada7
+        1ddf3204-1cdf-4314-b827-3e608fb5333c
+        44182d88-03fd-4392-aef1-cbaade65e671
+        a2e33687-555f-4b27-beef-a745c7dffbc4
+        bfb330a0-babd-48da-975c-74d11e53f7b7
+        d608f7ef-d3c2-43ae-8773-5599226a83da
+        eec17379-8fb4-453c-98b6-b65963b5a00b
+        f814decb-4a50-4625-99d9-4a5bf6398b85
+        f9bd3a55-273a-4d5d-963d-48589da56b59
       )
     )
