File: LF/LF.kicad_pcb (KiCad board)
At the start: 2 copper layers, 264 x 32 mm, 1 part

Commit message: Clean project
Parts:
- REF**: footprint CIS:CIS_Edge_Holes -> CIS:CIS_Edge_Holes_In
Other:
- outline, holes or cut-outs redrawn

Commit message: Update holes
Changed lines of the file:
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@@
         (effects (font (size 1 1) (thickness 0.15)))
     )
-    (pad "" thru_hole circle (at 3.5 -28.5) (size 4 4) (drill 3.1) (layers "*.Cu" "*.Mask"))
-    (pad "" thru_hole circle (at 3.5 -3.5) (size 4 4) (drill 3.1) (layers "*.Cu" "*.Mask"))
-    (pad "" thru_hole circle (at 88 -28.5) (size 4 4) (drill 3.1) (layers "*.Cu" "*.Mask"))
-    (pad "" thru_hole circle (at 88 -3.5) (size 4 4) (drill 3.1) (layers "*.Cu" "*.Mask"))
-    (pad "" thru_hole circle (at 176 -28.5) (size 4 4) (drill 3.1) (layers "*.Cu" "*.Mask"))
-    (pad "" thru_hole circle (at 176 -3.5287) (size 4 4) (drill 3.1) (layers "*.Cu" "*.Mask"))
-    (pad "" thru_hole circle (at 260.5 -28.5) (size 4 4) (drill 3.1) (layers "*.Cu" "*.Mask"))
-    (pad "" thru_hole circle (at 260.5 -3.5) (size 4 4) (drill 3.1) (layers "*.Cu" "*.Mask"))
-    (group "" (id efd7dfa4-ddc6-4e28-892f-13b9d91a71a3)
+    (pad "" thru_hole circle (at 3.5 -28.5) (size 4 4) (drill 3.2) (layers "*.Cu" "*.Mask"))
+    (pad "" thru_hole circle (at 3.5 -3.5) (size 4 4) (drill 3.2) (layers "*.Cu" "*.Mask"))
+    (pad "" thru_hole circle (at 88 -28.5) (size 4 4) (drill 3.2) (layers "*.Cu" "*.Mask"))
+    (pad "" thru_hole circle (at 88 -3.5) (size 4 4) (drill 3.2) (layers "*.Cu" "*.Mask"))
+    (pad "" thru_hole circle (at 176 -28.5) (size 4 4) (drill 3.2) (layers "*.Cu" "*.Mask"))
+    (pad "" thru_hole circle (at 176 -3.5287) (size 4 4) (drill 3.2) (layers "*.Cu" "*.Mask"))
+    (pad "" thru_hole circle (at 260.5 -28.5) (size 4 4) (drill 3.2) (layers "*.Cu" "*.Mask"))
+    (pad "" thru_hole circle (at 260.5 -3.5) (size 4 4) (drill 3.2) (layers "*.Cu" "*.Mask"))
+    (group "" (id 2887a8b2-aee5-40ea-818c-36717fd06432)
       (members
-        17283ed0-8005-494c-9ad5-9f186f01e515
-        7ca92d2a-8547-4826-9531-9dc215f92074
-        8aa04cc6-5a9e-4e5b-837f-5e35d512a7b2
-        8c941e19-64d0-4554-9842-a3cf032279fd
-        8dd00827-e86c-4ea6-8f60-50e94ebeaca5
-        9d9dcc87-45fc-47d2-a7c1-d6d63c72bc06
-        cd0c9901-132d-4528-81e8-8e0bf0816f9f
-        d4421c6c-597d-4969-baed-56777b64821e
-        fa86a7e1-92ef-492e-a033-8123d2fa2c38
+        1d67edfc-9e73-4822-8c30-2c8830163d84
+        2712df58-7a51-4c10-82e5-8aab5e9afd91
+        460ad9c7-8b5b-47bf-a61a-cac46489abdf
+        4a4494ad-481c-4786-af97-4851a09a8639
+        5187fa36-b4b0-4a94-9237-4556d9b238e3
+        7007b883-b8ff-4466-9eca-e5f831e9010d
+        8ad805c9-5662-49fa-b158-f4c7daad2e1c
+        e382c540-7a8f-477b-a151-d3acf8985a0d
+        f50854ba-3fe7-4a93-b377-ad247135a2a3
       )
     )
