File: LG/LG.kicad_pcb (KiCad board)
At the start: 2 copper layers, 264 x 32 mm, 4 parts

Commit message: Clean project
Parts:
- REF**: footprint CIS:CIS_Edge_Holes -> CIS:CIS_Edge_Holes_Out
Other:
- outline, holes or cut-outs redrawn

Commit message: Update holes
Parts:
- added REF**: VAL**, DVB_Connectors:PWR_PAD, F.Cu at (211.1, 109.0)
- added REF**: VAL**, DVB_Connectors:PWR_PAD, F.Cu at (192.9, 109.0)
- added REF**: VAL**, DVB_Connectors:PWR_PAD, F.Cu at (104.7, 109.0)
Other:
- outline, holes or cut-outs redrawn
